File: pcb/pcb.kicad_sch (KiCad schematic)
At the start: 118 parts, among them J1 Conn_02x20_JETSON, J10 Conn_01x02, J11 Conn_01x02, J12 Conn_01x02, J13 Conn_01x02, J14 Conn_01x02, J15 Conn_01x02, J16 Conn_01x02, J17 Conn_01x02, J18 Conn_01x04, J19 Conn_01x04, J2 Conn_02x22_STM32_LEFT, J2 Conn_02x22_STM32_RIGHT, J20 Conn_01x04, J21 Conn_01x04, J22 Conn_01x04, J23 Conn_01x04, J24 Conn_01x04, J25 Conn_01x04, J26 USB_B, J27 Conn_01x02, J28 Conn_02x22_Odd_Even_MountingP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, J29 Conn_02x22_Odd_Even_MountingP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, J3 Conn_24V, J31 Conn_ESC, J4 Conn_ESC, J5 Conn_Servo, J6 Conn_01x02, J7 Conn_01x02, J8 Conn_01x02, J9 Conn_01x02, Q1 NPN, SW1 SW_DIP_x01, U1 PCA9685PW, U2 CP2102N-Axx-xQFN20, U3 74AHC244, U4 MCP6002-xMS, U5 MCP6002-xMS, U6 MCP6002-xMS, U7 MCP6002-xMS, U8 4071

Commit message: chin
Parts:
- removed U8: 4071, symbol 4xxx:4071
- added J30, J41: ~, symbol Connector_Generic:Conn_02x03_Odd_Even
- added J50, J51, J52: ~, symbol Connector_Generic:Conn_01x02
- added J60, J70, J71: ~, symbol Connector_Generic:Conn_02x08_Odd_Even
- added J80: ~, symbol Connector_Generic:Conn_02x04_Odd_Even
- added Q2: NPN, symbol Simulation_SPICE:NPN
- added R41: R, symbol Device:R
- added U10: 4001, symbol 4xxx:4001
Connections:
- net BEC: now also J30.3 (Pin_3), J30.4 (Pin_4), J41.3 (Pin_3), J41.4 (Pin_4), J50.1 (Pin_1), Q2.1 (C), R41.2; no longer Q1.1 (C)
- net BTN7970_OUTPUT_0: now also J80.1 (Pin_1)
- net BTN7970_OUTPUT_1: now also J80.3 (Pin_3)
- net BTN7970_OUTPUT_2: now also J80.5 (Pin_5)
- net BTN7970_OUTPUT_3: now also J80.7 (Pin_7)
- net ESC_INPUT: now also J30.1 (Pin_1)
- net GND: now also Q1.3 (E), J30.5 (Pin_5), J30.6 (Pin_6), J41.5 (Pin_5), J41.6 (Pin_6), J50.2 (Pin_2), J51.2 (Pin_2), J52.2 (Pin_2), J70.12 (Pin_12), J70.16 (Pin_16), J70.4 (Pin_4), J70.8 (Pin_8), J71.12 (Pin_12), J71.16 (Pin_16), J71.4 (Pin_4), J71.8 (Pin_8), J80.2 (Pin_2), J80.4 (Pin_4), J80.6 (Pin_6), J80.8 (Pin_8)
- net Manual_Input: now also U10.3
- net PA4: now also J70.9 (Pin_9)
- net PA5: now also J70.11 (Pin_11)
- net PB10: now also J71.5 (Pin_5)
- net PB11: now also J71.7 (Pin_7)
- net PC2: now also J70.5 (Pin_5)
- net PC3: now also J70.7 (Pin_7)
- net PE0: now also J70.1 (Pin_1)
- net PE1: now also J70.3 (Pin_3)
- net PE6: now also J70.13 (Pin_13)
- net PE7: now also J70.15 (Pin_15)
- net S08: now also J71.1 (Pin_1)
- net S09: now also J71.3 (Pin_3)
- net S12: now also J71.9 (Pin_9)
- net S13: now also J71.11 (Pin_11)
- net S14: now also J71.13 (Pin_13)
- net S15: now also J71.15 (Pin_15)
- net SERVO_INPUT: now also J30.2 (Pin_2)
- net vrs_0: now also J60.1 (Pin_1)
- net vrs_1: now also J60.3 (Pin_3)
- net vrs_2: now also J60.5 (Pin_5)
- net vrs_3: now also J60.7 (Pin_7)
- net vrs_4: now also J60.9 (Pin_9)
- net vrs_5: now also J60.11 (Pin_11)
- net vrs_6: now also J60.13 (Pin_13)
- net vrs_7: now also J60.15 (Pin_15)
- net at R40.2: now also U10.1
- net at R39.1, SW1.2: now also U10.2
- net at J27.1 (Pin_1): now also Q2.3 (E); no longer Q1.3 (E)
- net PE9 renamed LCD_SWITCH
- new net: J60.10 (Pin_10), J60.12 (Pin_12), J60.14 (Pin_14), J60.2 (Pin_2), J60.4 (Pin_4), J60.6 (Pin_6), J60.8 (Pin_8)
- new net: Q1.1 (C), Q2.2 (B), R41.1
- new net -Vref: J60.16 (Pin_16)
- new net ESC_OUTPUT: J41.1 (Pin_1)
- new net SERVO_OUTPUT: J41.2 (Pin_2)
- new net V3.3: J52.1 (Pin_1), J70.10 (Pin_10), J70.14 (Pin_14), J70.2 (Pin_2), J70.6 (Pin_6), J71.10 (Pin_10), J71.14 (Pin_14), J71.2 (Pin_2), J71.6 (Pin_6)
- new net V5: J51.1 (Pin_1)
Other:
- moved on the sheet: J27, Q1
